File: arachne.kicad_sch (KiCad schematic)
At the start: 43 parts, among them J1 Leg1_coxa, J10 leg5_femur, J11 Leg6_coxa, J12 leg6_femur, J13 Conn_01x02, J14 Conn_01x03, J15 Conn_01x08_Socket, J16 Conn_01x15_Pin, J17 Conn_01x15_Pin, J18 sig, J19 USB_C_Receptacle_USB2.0_14P, J2 leg1_femur, J3 Leg2_coxa, J4 leg2_femur, J5 Leg3_coxa, J6 leg3_femur, J7 Leg4_coxa, J8 leg4_femur, J9 Leg5_coxa, SW1 RST/EN, SW2 BOOT, U1 ESP32-S3-WROOM-1, U2 PCA9685BS, U3 AMS1117-3.3, U4 HC-SR04

Commit message: Update PCB routing and KiCad project
Parts:
- removed C5: 1000u, symbol Device:C
- removed J14: Conn_01x03, symbol Connector_Generic:Conn_01x03
- removed J16, J17: Conn_01x15_Pin, symbol Connector:Conn_01x15_Pin
- removed J18: sig, symbol Connector:Conn_01x02_Pin
- added C8: 1000u, Capacitor_THT:C_Radial_D10.0mm_H12.5mm_P5.00mm, symbol Device:C
- added D2, D3: LED, LED_SMD:LED_0603_1608Metric, symbol Device:LED
- added D4: BAT60A, Diode_SMD:D_SOD-323, symbol Diode:BAT60A
- added J16: NEW_BUCK, Connector_PinHeader_2.54mm:PinHeader_2x02_P2.54mm_Vertical, symbol Connector_Generic:Conn_02x02_Top_Bottom
- added R6, R7: 330R, Resistor_SMD:R_0805_2012Metric, symbol Device:R
- C1, C2, C4, C6, C7: footprint (none) -> Capacitor_SMD:C_0805_2012Metric
- C3: footprint (none) -> Capacitor_SMD:C_1206_3216Metric
- D1: footprint digikey-footprints:SOT23-6L -> Package_TO_SOT_SMD:SOT-23-6
- F1: footprint (none) -> Fuse:Fuse_1206_3216Metric
- H1, H2, H3, H4: footprint (none) -> MountingHole:MountingHole_3.2mm_M3
- J1, J10, J11, J12, J2, J3, J4, J5, J6, J7, J8, J9: footprint (none) -> Connector_PinHeader_2.54mm:PinHeader_1x03_P2.54mm_Vertical
- J13: value Conn_01x02 -> BATTERY INPUT; footprint (none) -> TerminalBlock_Phoenix:TerminalBlock_Phoenix_MKDS-1,5-2-5.08_1x02_P5.08mm_Horizontal
- J15: value Conn_01x08_Socket -> MPU_PORT; footprint (none) -> Connector_PinHeader_2.54mm:PinHeader_1x08_P2.54mm_Vertical
- J19: footprint (none) -> Connector_USB:USB_C_Receptacle_HRO_TYPE-C-31-M-12
- R1, R2, R3, R4, R5: footprint (none) -> Resistor_SMD:R_0805_2012Metric
- SW1, SW2: footprint (none) -> Button_Switch_THT:SW_PUSH_6mm
Connections:
- net 5V is gone; now on net +5V: J1.2 (Pin_2), J10.2 (Pin_2), J11.2 (Pin_2), J12.2 (Pin_2), J2.2 (Pin_2), J3.2 (Pin_2), J4.2 (Pin_2), J5.2 (Pin_2), J6.2 (Pin_2), J7.2 (Pin_2), J8.2 (Pin_2), J9.2 (Pin_2)
- net +3.3V: now also R6.1
- net +5V: now also C8.1, R7.1; no longer J19.A4 (VBUS), J19.A9 (VBUS), J19.B4 (VBUS), J19.B9 (VBUS)
- net GND: now also D2.1 (K), D3.1 (K), J16.2 (Pin_2), J16.4 (Pin_4); no longer D1.5
- net 1: no longer names the net of U1.10 (IO17)
- net 10: no longer names the net of U1.34 (IO41)
- net 11: no longer names the net of U1.35 (IO42)
- net 12: no longer names the net of U1.26 (IO45)
- net 13: no longer names the net of U1.16 (IO46)
- net 14: no longer names the net of U1.24 (IO47)
- net 15: no longer names the net of U1.25 (IO48)
- net 16: no longer names the net of U1.9 (IO16)
- net 17: no longer names the net of U1.8 (IO15)
- net 18: no longer names the net of U1.22 (IO14)
- net 19: no longer names the net of U1.21 (IO13)
- net 2: no longer names the net of U1.11 (IO18)
- net 20: no longer names the net of U1.20 (IO12)
- net 21: no longer names the net of U1.19 (IO11)
- net 22: no longer names the net of U1.18 (IO10)
- net 23: no longer names the net of U1.17 (IO9)
- net 24: no longer names the net of U1.12 (IO8)
- net 25: no longer names the net of U1.7 (IO7)
- net 26: no longer names the net of U1.6 (IO6)
- net 27: no longer names the net of U1.15 (IO3)
- net 28: no longer names the net of U1.38 (IO2)
- net 29: no longer names the net of U1.39 (IO1)
- net 3: no longer names the net of U1.23 (IO21)
- net 4: no longer names the net of U1.28 (IO35)
- net 5: no longer names the net of U1.29 (IO36)
- net 6: no longer names the net of U1.30 (IO37)
- net 7: no longer names the net of U1.31 (IO38)
- net 8: no longer names the net of U1.32 (IO39)
- net 9: no longer names the net of U1.33 (IO40)
- net BAT_IN renamed +VIN
- net +VIN: now also J16.1 (Pin_1)
- net RX: no longer names the net of U1.36 (RXD0)
- net TX: no longer names the net of U1.37 (TXD0)
- new net: D2.2 (A), R6.2
- new net: D3.2 (A), R7.2
- new net: D4.1 (K), J19.A4 (VBUS), J19.A9 (VBUS), J19.B4 (VBUS), J19.B9 (VBUS)
- new net +VOUT: C8.2, J16.3 (Pin_3)
- new net VBUS: D1.5, D4.2 (A)
- no-connect marks 10 -> 40
