File: arachne.kicad_pcb (KiCad board)
At the start: 2 copper layers, 80 x 100 mm, 45 parts, among them J1 Leg1_coxa, J10 leg5_femur, J11 Leg6_coxa, J12 leg6_femur, J13 BATTERY INPUT, J15 MPU_PORT, J16 NEW_BUCK, J19 USB_C_Receptacle_USB2.0_14P, J2 leg1_femur, J3 Leg2_coxa, J4 leg2_femur, J5 Leg3_coxa, J6 leg3_femur, J7 Leg4_coxa, J8 leg4_femur, J9 Leg5_coxa, SW1 RST/EN, SW2 BOOT, U1 ESP32-S3-WROOM-1, U2 PCA9685BS, U3 AMS1117-3.3, U4 HC-SR04

Commit message: kicad_arachne
Routing:
- net /Trig: track 0.53 -> 168.9 mm
- net +3.3V: track 110.7 -> 44.5 mm
- net GND: track 75.3 -> 17.2 mm, vias 3 -> 0
- net +5V: track 134.8 -> 160.4 mm
- removed copper zone on B.Cu, net GND
Other:
- board text added: "${REFERENCE}"

Commit message: Update PCB routing and project files
Parts:
- moved D1 17.9 mm to (70.4, 74.5)
- moved C3 17.9 mm to (86.0, 90.5)
- moved R3 17.9 mm to (94.4, 134.5)
- moved U3 17.9 mm to (84.8, 81.0)
- moved J10 17.9 mm to (130.8, 105.4)
- moved J11 17.9 mm to (130.8, 93.4)
- moved J12 17.9 mm to (130.8, 81.4)
- moved J3 17.9 mm to (58.0, 98.8)
- moved J9 17.9 mm to (130.8, 117.4)
- moved C7 17.9 mm to (89.8, 62.8)
- moved C1 17.9 mm to (92.3, 67.8)
- moved C2 17.9 mm to (75.5, 82.0)
- moved C4 17.9 mm to (110.5, 114.0)
- moved C6 17.9 mm to (82.5, 102.5)
- moved C8 17.9 mm to (78.5, 128.5)
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Routing:
- net GND: track 17.2 -> 412.8 mm, vias 0 -> 19
- net +5V: track 160.4 -> 336.8 mm, vias 0 -> 13
- net /echo_final: track 5.16 -> 76.5 mm, vias 0 -> 2
- net +3.3V: track 44.5 -> 105.4 mm, vias 0 -> 5
- net /EN: track 17.5 -> 50.9 mm, vias 0 -> 2
- net /D-: track 8.65 -> 24.5 mm, vias 0 -> 2
- net Net-(J13-Pin_1): track 0.00 -> 15.0 mm, vias 0 -> 2
- net Net-(D4-K): track 7.01 -> 15.6 mm, vias 0 -> 2
- net /D+: track 8.81 -> 13.7 mm, vias 0 -> 2
- net Net-(J19-CC2): track 6.48 -> 8.62 mm
- added copper zone on B.Cu, net GND
Other:
- outline, holes or cut-outs redrawn
- board text removed: "${REFERENCE}"
